File: Onion_O2S_mPCIe.sch (EAGLE design)
At the start: 7 parts, among them J1 693071020811, U1 ONION_OMEGA2S

Commit message: continued layout
Parts:
- added LED1: (no value), led:LEDCHIPLED_0603
- added R1: (no value), rcl:R-EU_R0603
Connections:
- new net N$1: LED1.C, R1.2
- net !WLED: now also R1.1
- net +3V3: now also LED1.A
Changed lines of the file:
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@@
 <part name="J1" library="Wurth_Connectors_WR-CRD" library_urn="urn:adsk.eagle:library:16444847" deviceset="693071020811" device="" package3d_urn="urn:adsk.eagle:package:16444883/5" value="693071020811"/>
 <part name="U$1" library="Eigene-Rietig" library_urn="urn:adsk.eagle:library:40964436" deviceset="MINI_PCIE" device="" package3d_urn="urn:adsk.eagle:package:43484125/3"/>
+<part name="LED1" library="led" library_urn="urn:adsk.eagle:library:259" deviceset="LED" device="CHIPLED_0603" package3d_urn="urn:adsk.eagle:package:15822/2"/>
+<part name="R1" library="rcl" library_urn="urn:adsk.eagle:library:44894963" deviceset="R-EU_" device="R0603" package3d_urn="urn:adsk.eagle:package:23555/3"/>
+<part name="+3V5" library="supply1" library_urn="urn:adsk.eagle:library:371" deviceset="+3V3" device=""/>
 </parts>
 <sheets>
@@
 <attribute name="NAME" x="210.82" y="146.05" size="1.778" layer="95"/>
 <attribute name="VALUE" x="210.82" y="71.12" size="1.778" layer="96"/>
+</instance>
+<instance part="LED1" gate="G$1" x="182.88" y="220.98" smashed="yes">
+<attribute name="NAME" x="186.436" y="216.408" size="1.778" layer="95" rot="R90"/>
+<attribute name="VALUE" x="188.595" y="216.408" size="1.778" layer="96" rot="R90"/>
+</instance>
+<instance part="R1" gate="G$1" x="182.88" y="208.28" smashed="yes" rot="R90">
+<attribute name="NAME" x="181.3814" y="204.47" size="1.778" layer="95" rot="R90"/>
+<attribute name="VALUE" x="186.182" y="204.47" size="1.778" layer="96" rot="R90"/>
+</instance>
+<instance part="+3V5" gate="G$1" x="182.88" y="228.6" smashed="yes">
+<attribute name="VALUE" x="180.34" y="223.52" size="1.778" layer="96" rot="R90"/>
 </instance>
 </instances>
@@
 <label x="261.62" y="132.08" size="1.27" layer="95" xref="yes"/>
 <pinref part="U$1" gate="G$1" pin="LED_WLAN"/>
+</segment>
+<segment>
+<pinref part="R1" gate="G$1" pin="1"/>
+<wire x1="182.88" y1="203.2" x2="182.88" y2="190.5" width="0.1524" layer="91"/>
+<wire x1="182.88" y1="190.5" x2="170.18" y2="190.5" width="0.1524" layer="91"/>
+<label x="170.18" y="190.5" size="1.27" layer="95" rot="R180" xref="yes"/>
 </segment>
 </net>
@@
 <wire x1="312.42" y1="284.48" x2="312.42" y2="299.72" width="0.1524" layer="91"/>
 </segment>
+<segment>
+<pinref part="+3V5" gate="G$1" pin="+3V3"/>
+<pinref part="LED1" gate="G$1" pin="A"/>
+<wire x1="182.88" y1="226.06" x2="182.88" y2="223.52" width="0.1524" layer="91"/>
+</segment>
 </net>
 <net name="UART0_TX" class="0">
@@
 </segment>
 </net>
+<net name="N$1" class="0">
+<segment>
+<pinref part="LED1" gate="G$1" pin="C"/>
+<pinref part="R1" gate="G$1" pin="2"/>
+<wire x1="182.88" y1="215.9" x2="182.88" y2="213.36" width="0.1524" layer="91"/>
+</segment>
+</net>

Commit message: * Completely changed pinout * Started Eval Board
Parts:
- added LED2: (no value), led:LEDCHIPLED_0603
- added Q2: 5.8A/30V/35mΩ, SparkFun-DiscreteSemi:MOSFET-NCH-AO3404A
- added Q3: BC807-16SMD, transistor-pnp:BC807-16SMD
- added R2: (no value), rcl:R-EU_R0603
- added R3, R9: 10k, rcl:R-EU_R0603
- added R4, R5: 0R, rcl:R-EU_R0603
- renumbered U$1 to EDGECON1
Connections:
- removed net ETH0_RXI_P: EDGECON1.+3V3AUX@24, U1.RXI_P0
- removed net ETH0_TXO_P: EDGECON1.GND@21, U1.TXO_P0
- removed net USB_D_P: EDGECON1.USB_D+, U1.USB_DP
- new net !HW_RST: EDGECON1.+1V5@48, Q2.G, U1.!HW_RST
- new net !PERST: EDGECON1.RSVRD51, U1.GPIO_36/!PERST
- new net ETH0_RXI_+: EDGECON1.WAKE, U1.RXI_P0
- new net ETH0_TXO_+: EDGECON1.COEX2, U1.TXO_P0
- new net LED: R2.1, U1.GPIO_11
- new net N$2: Q3.B, R9.2
- new net N$3: Q2.D, R9.1
- new net N$4: Q3.C, R3.2, R4.1, R5.2
- new net N$7: LED2.C, R2.2
- new net SPI_CLK: EDGECON1.SMB_DATA, U1.SPI_CLK
- new net SPI_CS0: EDGECON1.+1V5@28, U1.SPI_CS0
- new net SPI_CS1: EDGECON1.PETP0, U1.SPI_CS1/GPIO6
- new net SPI_MISO: EDGECON1.PETN0, U1.SPI_MISO
- new net SPI_MOSI: EDGECON1.SMB_CLK, U1.SPI_MOSI
- new net SW_RST: EDGECON1.RSVRD49, U1.GPIO_38/SW_RST
- new net USB_D_+: EDGECON1.REFCLK+, U1.USB_DP
- new net VDD_FLASH: R5.1, U1.VDD_FLASH
- net !WLED: now also EDGECON1.RSVRD47; no longer EDGECON1.LED_WLAN
- net +3V3: now also LED2.A, Q3.E, R4.2; no longer EDGECON1.GND@4, EDGECON1.GND@50
- net ETH0_RXI_N: now also EDGECON1.COEX1; no longer EDGECON1.PERST
- net ETH0_TXO_N: now also EDGECON1.CLKREQ; no longer EDGECON1.PERN0
- net GND: now also EDGECON1.GND@15, EDGECON1.GND@18, EDGECON1.GND@21, EDGECON1.GND@26, EDGECON1.GND@27, EDGECON1.GND@29, EDGECON1.GND@34, EDGECON1.GND@35, EDGECON1.GND@37, EDGECON1.GND@4, EDGECON1.GND@40, EDGECON1.GND@43, EDGECON1.GND@50, EDGECON1.GND@9, EDGECON1.HOLES, Q2.S, R3.1; no longer EDGECON1.COEX1, EDGECON1.RSVRD49, EDGECON1.RSVRD51, EDGECON1.WAKE
- net GPIO_14: now also EDGECON1.PERN0; no longer EDGECON1.GND@26
- net GPIO_15: now also EDGECON1.PERST; no longer EDGECON1.+1V5@28
- net GPIO_16: now also EDGECON1.W_DISABLE; no longer EDGECON1.GND@27
- net GPIO_17: now also EDGECON1.UIM_C4; no longer EDGECON1.PERP0
- net GPIO_18: now also EDGECON1.UIM_C8; no longer EDGECON1.GND@29
- net GPIO_19: now also EDGECON1.UIM_VPP; no longer EDGECON1.PETN0
- net GPIO_20: now also EDGECON1.UIM_RESET; no longer EDGECON1.SMB_DATA
- net GPIO_21: now also EDGECON1.UIM_CLK; no longer EDGECON1.SMB_CLK
- net I2C_SCK: now also EDGECON1.USB_D+; no longer EDGECON1.RSVRD47
- net I2C_SDA: now also EDGECON1.USB_D-; no longer EDGECON1.+1V5@48
- net I2S_SDI: now also EDGECON1.LED_WLAN; no longer EDGECON1.+3V3AUX@41
- net I2S_SDO: now also EDGECON1.LED_WWAN; no longer EDGECON1.GND@43
- net I2S_WS: now also EDGECON1.+3V3AUX@41; no longer EDGECON1.GND@40
- net UART0_RX: now also EDGECON1.+3V3AUX@24; no longer EDGECON1.W_DISABLE
- net UART0_TX: now also EDGECON1.PERP0; no longer EDGECON1.GND@18
- net UART1_RX: now also EDGECON1.RSVRD45; no longer EDGECON1.GND@9
- net UART1_TX: now also EDGECON1.LED_WPAN; no longer EDGECON1.UIM_DATA
- net USB_D_N: now also EDGECON1.REFCLK-; no longer EDGECON1.USB_D-
Other:
- moved on the sheet: C1, C2, J1

Commit message: - small changes to the sikscreen of the module - continued design of Eval Board
Other:
- moved on the sheet: C1, C2, EDGECON1, J1, LED2, Q2, Q3, R2, R3, R4, R5, R9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
