File: Eval_Board/Onion_PCIe_Eval.sch (EAGLE design)
At the start: 7 parts, among them J1 61400416021, J2 7499010211A, J3 629722000214, Q1 LORA_MPCIE

Commit message: - small changes to the sikscreen of the module - continued design of Eval Board
Parts:
- removed D1: 82400102 5V, Wurth_EMC Components_WE-TVS:WE-TVS-HS_SOT23-6L_82400102
- removed Q1: LORA_MPCIE, Eigene-Rietig:LORA_MPCIE
- added D2, D3: 82400102 5V, Wurth_EMC Components_WE-TVS:WE-TVS-HS_SOT23-6L_82400102
- added R1, R2, R3, R4: 5k1, rcl:R-EU_R0603
- added U$1: ONION_OMEGA2S_MPCIE, Eigene-Rietig:ONION_OMEGA2S_MPCIE
- added U1: FT230XS, Eigene-Rietig:FT230XS
Connections:
- new net CONSOLE_RXD: U$1.GPIO_13/UART_RXD0, U1.TXD
- new net CONSOLE_TXD: U$1.GPIO_12/UART_TXD0, U1.RXD
- new net ETH_RX_N: J2.RD+, R2.2, U$1.RXI_N0
- new net ETH_RX_P: J2.RD-, R1.2, U$1.RXI_P0
- new net ETH_TX_N: J2.TD+, R4.1, U$1.TXO_N0
- new net ETH_TX_P: J2.TD-, R3.1, U$1.TXO_P0
- new net N$1: R1.1, R2.1
- new net N$3: R3.2, R4.2
- new net N$4: U1.!RESET, U1.3V3OUT, U1.VCCIO
- new net USB_DN_N: D2.I/O3, U$1.USB_DM
- new net USB_DN_P: D2.I/O4, U$1.USB_DP
- new net USB_DN_PROT_N: D2.I/O1, J1.D-
- new net USB_DN_PROT_P: D2.I/O2, J1.D+
- net +5V: now also D2.VDD, D3.VDD, U1.VCC; no longer D1.VDD
- net GND: now also D2.GND, D3.GND, U$1.GND, U1.GND; no longer D1.GND
- net USB_D_N: now also D3.I/O1; no longer D1.I/O2
- net USB_D_P: now also D3.I/O2; no longer D1.I/O1
- net USB_D_PROT_N: now also D3.I/O3, U1.USBDP; no longer D1.I/O4
- net USB_D_PROT_P: now also D3.I/O4, U1.USBDM; no longer D1.I/O3
Other:
- moved on the sheet: J1, J3, R6, R9
